File: Eagle CAD/audio sw - daughter.sch (EAGLE design)
At the start: 61 parts, among them J1 DCJ0202PIN, J2 3.5MM-J3SJI-353, J3 3.5MM-J3SJI-353, J4 3.5MM-J3SJI-353, J5 PN87520-S, J7 PINHD-1X8, U1 BUCK4_THRU, U2 LM340LZ-05, U5 STM32F030F4P6, U6 XC6206P332MR, X1 12MHz

Commit message: Tweaks for daughtercard Hardware updates
Parts:
- removed $1_40_$: CC-BY-NC100%, Misc logo:CC-BY-NC100%
- removed C10, C11, C15, C18, C9: 0.1uF, ipc-7351-capacitor:CAPACITOR_0603
- removed C12, C13: 22pF, ipc-7351-capacitor:CAPACITOR_0603
- removed C14, C16, C17, C20: 1uF, ipc-7351-capacitor:CAPACITOR_0603
- removed C19: 10uF, ipc-7351-capacitor:CAPACITOR_0805
- removed C21, C22, C23, C24, C25: 1n8, ipc-7351-capacitor:CAPACITOR_0603
- removed D1: (no value), ipc-7351-diode:KA2KA_SOT-23
- removed J1: DCJ0202PIN, Misc Conn:DCJ0202PIN
- removed J2, J3, J4: 3.5MM-J3SJI-353, Misc Conn:3.5MM-J3SJI-353
- removed J5: PN87520-S, con-berg:PN87520-S
- removed J6: (no value), Misc Conn:PINHD-1X4_2.54
- removed J7: PINHD-1X8, Misc Conn:PINHD-1X8
- removed J8: (no value), Misc Conn:PINHD-1X3
- removed J9: (no value), Misc Conn:PINHD-1X2_2.54
- removed L3: 600R, ipc-7351-resistor:RESISTOR_0805
- removed RN1: 10Kx5, SparkFun-Passives:RPACK-BUSSED-SIP-PTH-5
- removed S1: (no value), SparkFun-Electromechanical:TAC_SWITCHPTH
- removed U$1: POLARITY, Misc logo:POLARITY
- removed U4: (no value), Misc opto:AX-1838HS
- removed U5: STM32F030F4P6, Misc Processor:STM32F030F4P6
- removed U6: XC6206P332MR, Misc Power:MCP1700/TT
- removed X1: 12MHz, crystal:CRYSTALHC49U-V
- added LICENSE1: CC-BY-NC100%, Misc logo:CC-BY-NC100%
- added R11, R12, R13, R14, R15, R16, R17, R18, R19, R20, R21, R22, R23, R24, R27: 10K, ipc-7351-resistor:RESISTOR_0603
- added R25: 1K, ipc-7351-resistor:RESISTOR_0603
- added R26, R28: 4K7, ipc-7351-resistor:RESISTOR_0603
- C1, JP1, JP2, R5, R6, R7, R8: PARTNO * -> (none)
- C2: device ipc-7351-capacitor:CAPACITOR_0805 -> ipc-7351-capacitor:CAPACITOR_0603; PARTNO * -> (none)
- C3: value 470uF/25V -> 0.1uF; device Misc Passives:CAP_POLPTH3 -> ipc-7351-capacitor:CAPACITOR_0603; PARTNO * -> (none)
- C4, C5: value 1uF -> 0.1uF; PARTNO * -> (none)
- C6: value 47uF/25V -> 0.1uF; device Misc Passives:CAP_POLPTH2 -> ipc-7351-capacitor:CAPACITOR_0603; PARTNO * -> (none)
- C7: value 1uF -> 22uF; device ipc-7351-capacitor:CAPACITOR_0603 -> ipc-7351-capacitor:POLARISED_C_CASE; PARTNO * -> (none)
- C8: value 470uF/25V -> 22uF; device Misc Passives:CAP_POLPTH3 -> ipc-7351-capacitor:POLARISED_C_CASE; PARTNO * -> (none)
- L1, L2: value 600R -> 600Z; PARTNO * -> (none)
- R1, R4: value 10K -> 4K7; PARTNO * -> (none)
- R10: value NC-0R -> 10K; device ipc-7351-resistor:RESISTOR_0805 -> ipc-7351-resistor:RESISTOR_0603; PARTNO * -> (none)
- R2: value NC-0R -> 4K7; PARTNO * -> (none)
- R3: value 475R -> 4K7; PARTNO * -> (none)
- R9: value 0R -> 10K; device ipc-7351-resistor:RESISTOR_0805 -> ipc-7351-resistor:RESISTOR_0603; PARTNO * -> (none)
- U1: value BUCK4_THRU -> NE5532N; device Misc Power:BUCK4_THRU -> linear:LM358D; PARTNO * -> (none)
- U2: value LM340LZ-05 -> NE5532N; device linear:LM340LZ-05 -> linear:LM358D; PARTNO * -> (none)
- U3: value (none) -> 74HC4052PW; device linear:79L05Z -> Misc Logic:4052PW; PARTNO * -> (none)
Connections:
- removed net !RST: C11.2, J7.P$1, U5.!RST
- removed net +3.3V: C14.2, C15.2, C17.2, C18.2, C20.2, J6.4, J7.P$6, R2.2, RN1.1, U4.VCC, U5.VDD, U5.VDDA, U6.VO
- removed net +5V_SMPS: C8.+, J5.1, J8.1, L3.2, U1.VO
- removed net /LED: J7.P$7, R2.1, R3.2
- removed net D/!C: J7.P$3, U5.PA6/MISO
- removed net IR: U4.OUT, U5.PB1
- removed net MOSI: J7.P$4, U5.PA7/MOSI
- removed net N$14: J3.2, JP1.4
- removed net N$15: J3.1, JP1.6, R10.1
- removed net N$19: J3.5, JP1.5
- removed net N$22: C5.2, L1.1, U2.VI
- removed net N$23: R8.1, S1.1, S1.2
- removed net N$25: C6.+, C7.2, L2.1, U3.VI
- removed net N$27: C1.1, D1.KA
- removed net N$29: C4.2, D1.A, L2.2
- removed net N$32: R1.2, U5.BOOT0
- removed net N$36: C21.2, R5.2, RN1.2, U5.PA0
- removed net N$37: C22.2, R7.2, RN1.3, U5.PA1
- removed net N$38: C23.2, R4.2, RN1.4, U5.PA2/TXD
- removed net N$39: C24.2, R6.2, RN1.5, U5.PA3/RXD
- removed net N$40: C25.2, J9.1, R8.2, RN1.6, U5.PA4/NSS
- removed net N$41: C13.2, U5.PF0/OSC_IN, X1.1
- removed net N$42: C12.2, U5.PF1/OSC_OUT, X1.2
- removed net SCK: J7.P$5, U5.PA5/SCK
- removed net SWCLK: J6.1, U5.PA14/SWCLK
- removed net SWDIO: J6.3, U5.PA13/SWDIO
- removed net U1_SW: C1.2
- removed net VIN: C2.2, C3.+, J1.1, J8.3, L1.2, U1.VI
- new net GND0: JP1.3, R1.1, R3.1, R5.1, R6.1
- new net GND1: JP1.6, R2.1, R4.1, R7.1, R8.1
- new net L0_IN: JP1.2, R10.1, R3.2
- new net L1_IN: JP1.5, R12.1, R4.2
- new net N$10: JP2.6, L2.1
- new net N$11: R11.2, R15.2, U2A.+IN
- new net N$12: R19.1, R7.2, U2A.-IN
- new net N$13: R24.2, U3A.Y2
- new net N$16: R12.2, R16.2, U2B.+IN
- new net N$17: R20.1, R8.2, U2B.-IN
- new net N$2: R17.1, R5.2, U1A.-IN
- new net N$3: C6.2, R25.2, R27.2, U3P.VCC
- new net N$6: R10.2, R14.2, U1B.+IN
- new net N$7: R18.1, R6.2, U1B.-IN
- new net N$8: JP2.4, L1.1
- new net R0_IN: JP1.1, R1.2, R9.1
- new net R1_IN: JP1.4, R11.1, R2.2
- net +5V: now also C1.2, C3.2, C7.+, L1.2, R25.1, U1P.V+, U2P.V+; no longer C9.2, JP2.4, U2.VO
- net -5V: now also C2.2, C4.2, C5.2, C8.-, L2.2, U1P.V-, U2P.V-, U3P.VEE; no longer C10.2, JP2.6, U3.VO
- net AGND: now also C1.1, C3.1, C6.1, C7.-, C8.+, R13.1, R14.1, R15.1, R16.1, R26.1, R27.1, R28.1, U3A.INH, U3P.GND; no longer C10.1, C11.1, C12.1, C13.1, C14.1, C15.1, C16.1, C17.1, C18.1, C19.1, C20.1, C21.1, C22.1, C23.1, C24.1, C25.1, C3.-, C6.-, C7.1, C8.-, C9.1, D1.K, J1.2, J1.3, J4.1, J5.4, J5.S1, J5.S2, J6.2, J7.P$2, J7.P$8, J8.2, J9.2, R1.1, R10.2, R3.1, R9.2, S1.3, S1.4, U1.GND, U2.GND, U3.GND, U4.GND, U5.VSS, U6.GND
- net CTRL0: now also U3A.A; no longer U5.PA9/SCL
- net CTRL1: now also U3A.B; no longer U5.PA10/SDA
- net L0: now also R18.2, R22.1, U1B.OUT, U3A.X0; no longer R6.1
- net L1: now also R20.2, R21.1, U2B.OUT, U3A.X1; no longer R7.1
- net L_OUT: now also R28.2, U3A.X; no longer J4.5
- net N$1: now also R13.2, R9.2, U1A.+IN; no longer C16.2, C19.2, L3.1, U6.VI
- net N$4: now also R22.2, U3A.X3; no longer J2.2, JP1.1
- net N$5: now also R21.2, U3A.X2; no longer J2.1, JP1.3, R9.1
- net N$9: now also R23.2, U3A.Y3; no longer J2.5, JP1.2
- net R0: now also R17.2, R24.1, U1A.OUT, U3A.Y0; no longer R4.1
- net R1: now also R19.2, R23.1, U2A.OUT, U3A.Y1; no longer R5.1
- net R_OUT: now also R26.2, U3A.Y; no longer J4.2
Other:
- note added: "VIH = 0.7V*Vcc(max), 0.5*Vcc (typ) VCC to 4.5V -> VIH = 3.15V"
- note removed: "Analog Daughter card"
- note removed: "Aux. Power"
- note removed: "Buck converter Switching node"
- note removed: "DC: 9V-18V >7W"
- note removed: "External buttons"
- note removed: "Grounding Option"
- note removed: "IR Receiver"
- note removed: "LCD (Nokia 5510)"
- note removed: "Polarity select"
- note removed: "SWD Hardware Debugger"
- moved on the sheet: C1, C2, C4, C5, JP1, JP2, L1, L2, R1, R10, R2, R3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
