File: Eagle CAD/audio sw.brd (EAGLE design)
At the start: 67.3 x 47 mm, 60 parts, among them J1 DCJ0202PIN, J2 3.5MM-J3SJI-353, J3 3.5MM-J3SJI-353, J4 3.5MM-J3SJI-353, J5 PN87520-S, J7 PINHD-1X8, U1 BUCK4_THRU, U2 LM340LZ-05, U5 STM32F030F4P6, U6 MCP1700/TT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

Commit message: Relay version - added Audio switching, bug fixes, updates Minor tweak for noisy relay circuit Bug fix - wrong define constants used.  :( Change alti-alias filter to 18kHz + cleanup Update CAD files Update simulation file
Parts:
- U2, U3: device linear:TO92 -> linear:TO92-CLP
Changed lines of the file:
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@@
 <setting verticaltext="up"/>
 </settings>
-<grid distance="0.05" unitdist="inch" unit="inch" style="lines" multiple="1" display="no" altdistance="0.005" altunitdist="inch" altunit="inch"/>
+<grid distance="0.05" unitdist="inch" unit="mm" style="lines" multiple="1" display="no" altdistance="0.005" altunitdist="inch" altunit="inch"/>
 <layers>
 <layer number="1" name="Top" color="4" fill="1" visible="yes" active="yes"/>
@@
 <layer number="41" name="tRestrict" color="4" fill="10" visible="yes" active="yes"/>
 <layer number="42" name="bRestrict" color="1" fill="10" visible="yes" active="yes"/>
-<layer number="43" name="vRestrict" color="2" fill="10" visible="yes" active="yes"/>
+<layer number="43" name="vRestrict" color="2" fill="10" visible="no" active="yes"/>
 <layer number="44" name="Drills" color="7" fill="1" visible="no" active="yes"/>
 <layer number="45" name="Holes" color="7" fill="1" visible="no" active="yes"/>
@@
 <layer number="220" name="220bmp" color="21" fill="1" visible="no" active="no"/>
 <layer number="221" name="221bmp" color="22" fill="1" visible="no" active="no"/>
-<layer number="222" name="222bmp" color="23" fill="1" visible="no" active="no"/>
 <layer number="223" name="223bmp" color="24" fill="1" visible="no" active="no"/>
 <layer number="224" name="224bmp" color="25" fill="1" visible="no" active="no"/>
@@
 <attribute name="VALUE" x="31.115" y="29.591" size="1.27" layer="27" rot="R270"/>
 </element>
-<element name="U2" library="linear" package="TO92" value="LM340LZ-05" x="41.402" y="29.21" smashed="yes" rot="R90">
+<element name="U2" library="linear" package="TO92-CLP" value="LM340LZ-05" x="41.402" y="29.21" smashed="yes" rot="R90">
 <attribute name="NAME" x="44.577" y="30.353" size="0.6096" layer="25" ratio="15" rot="R180"/>
 <attribute name="VALUE" x="42.672" y="32.131" size="0.4064" layer="27" ratio="10" rot="R90"/>
@@
 <attribute name="VALUE" x="42.594" y="33.6565" size="0.4064" layer="28" font="vector" ratio="10" rot="MR180"/>
 </element>
-<element name="U3" library="linear" package="TO92" value="" x="40.767" y="22.987" smashed="yes" rot="R270">
+<element name="U3" library="linear" package="TO92-CLP" value="" x="40.767" y="22.987" smashed="yes" rot="R270">
 <attribute name="NAME" x="42.926" y="20.447" size="0.6096" layer="25" ratio="15"/>
 <attribute name="VALUE" x="39.497" y="20.066" size="1.27" layer="27" ratio="10" rot="R270"/>

Commit message: Tweaks for daughtercard Hardware updates
Parts:
- added R10: NC-0R, ipc-7351-resistor:RESC2012X70N
- added R9: 0R, ipc-7351-resistor:RESC2012X70N
- C21, C22, C23, C24, C25: value 2n2 -> 1n8
- U6: value MCP1700/TT -> XC6206P332MR
Connections:
- net AGND: now also R10.2, R9.2
- net N$15: now also R10.1
- net N$5: now also R9.1
Routing:
- net N$5: track 28.2 -> 30.7 mm
- net N$15: track 46.6 -> 49.0 mm
