File: Eagle CAD/audio sw - daughter - rev 0.1.brd (EAGLE design)
At the start: 35.6 x 15.2 mm, 44 parts, among them U4 NE5532N, U5 NE5532N, U6 74HC4052PW

Commit message: Enable Loudness Protection + BOM Consolidation
Parts:
- C1, C2: value 22uF -> 22uF/16V
- R21, R22, R23, R24: value 3K92 -> 4K7
- R25, R26, R27, R28: value 20K -> 10K
- R29, R30: value 10K -> 4K7
