File: Eagle CAD/audio sw - daughter - rev 0.1.sch (EAGLE design)
At the start: 44 parts, among them U4 NE5532N, U5 NE5532N, U6 74HC4052PW

Commit message: Enable Loudness Protection + BOM Consolidation
Parts:
- C1, C2: value 22uF -> 22uF/16V; PARTNO (none) -> *
- C10, C5, C6, C7, C8, C9, JP1, JP2, LICENSE1, R1, R10, R11, R12, R13, R14, R15, R16, R17, R18, R19, R2, R20, R3, R4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: PARTNO (none) -> *
- R21, R22, R23, R24: value 3K92 -> 4K7; PARTNO (none) -> *
- R25, R26, R27, R28: value 20K -> 10K; PARTNO (none) -> *
- R29, R30: value 10K -> 4K7; PARTNO (none) -> *
